Commit message: gpt + cline did a good job in writing the xacro

File: models/urdf/orcahand.urdf.xacro (robot description, xacro)
@@ -24,5 +24,5 @@
       </inertial>
       <visual name="visual_tower_main_mesh">
-         <origin xyz="${s * 0.04069509610470536} -0.00012511806280993186 0.02312294830988657" rpy="${s * -0.007252153364137093} -0.004356332895580239 1.533990149039079"/>
+         <origin xyz="${s * 0.04069509610470536} -0.00012511806280993186 0.02312294830988657" rpy="${s * -0.007252153364137093} -0.004356332895580239 ${'1.6076025045507145' if chirality == 'left' else '1.533990149039079'}"/>
          <geometry>
             <mesh filename="${rospackage_path}/visual/tower_main_mesh.stl"/>
@@ -31,5 +31,5 @@
       </visual>
       <collision name="collision_tower_main_mesh">
-         <origin xyz="${s * 0.04102610596606573} 0.0008755408110132971 0.03758955025925282" rpy="0.0663641604020242 ${s * 0.10532695421927696} ${s * -0.7765909134463538}"/>
+         <origin xyz="${s * 0.04102610596606573} 0.0008755408110132971 0.03758955025925282" rpy="0.0663641604020242 ${-s * 0.10532695421927696} ${s * -0.7765909134463538}"/>
          <geometry>
             <mesh filename="${rospackage_path}/collision/tower_main_mesh.stl"/>
@@ -38,5 +38,5 @@
       </collision>
       <visual name="visual_tower_hull_mesh">
-         <origin xyz="${s * 0.04062006698890873} -3.726678941555769e-06 0.009339292204050375" rpy="1.5694791585075034 0.00015194814647356836 -0.0006505124711437826"/>
+         <origin xyz="${'-0.040379932753305224 -3.7268131082661286e-06 0.009339292178809312' if chirality == 'left' else '0.04062006698890873 -3.726678941555769e-06 0.009339292204050375'}" rpy="${'1.5694791593330333 0.00015194626808745504 -0.0006505202080002714' if chirality == 'left' else '1.5694791585075034 0.00015194814647356836 -0.0006505124711437826'}"/>
          <geometry>
             <mesh filename="${rospackage_path}/visual/tower_hull_mesh.stl"/>
@@ -45,5 +45,5 @@
       </visual>
       <collision name="collision_tower_hull_mesh">
-         <origin xyz="${s * 0.04061884697236149} 7.083739226185091e-06 0.009306225228503611" rpy="1.5691929949477865 -6.931644826568828e-05 -0.0012916867662787768"/>
+         <origin xyz="${'-0.04038115277822704 7.083580336650913e-06 0.009306225237370189' if chirality == 'left' else '0.04061884697236149 7.083739226185091e-06 0.009306225228503611'}" rpy="${'1.5691929968226592 -6.931705689772194e-05 -0.001291690818031932' if chirality == 'left' else '1.5691929949477865 -6.931644826568828e-05 -0.0012916867662787768'}"/>
          <geometry>
             <mesh filename="${rospackage_path}/collision/tower_hull_mesh.stl"/>
@@ -52,5 +52,5 @@
       </collision>
       <visual name="visual_tower_text_mesh">
-         <origin xyz="${s * 0.040617526582081696} 4.362558106779257e-06 0.02737731026837054" rpy="8.992806499463768e-14 -1.570241143557443 1.5988186561911613"/>
+         <origin xyz="${'-0.04038247369298952 4.361834990936047e-06 0.027377310183930685' if chirality == 'left' else '0.040617526582081696 4.362558106779257e-06 0.02737731026837054'}" rpy="${'-5.88418203051333e-14 -1.5702411380021881 1.598818649875384' if chirality == 'left' else '8.992806499463768e-14 -1.570241143557443 1.5988186561911613'}"/>
          <geometry>
             <mesh filename="${rospackage_path}/visual/tower_text_mesh.stl"/>
@@ -58,4 +58,11 @@
          <material name="white"/>
       </visual>
+      <collision name="collision_tower_text_mesh">
+         <origin xyz="${'-0.04031654534641286 -0.0011250821606647178 0.027716099560264867' if chirality == 'left' else '0.04068345506360967 -0.0011250828560853416 0.027716099517902396'}" rpy="${'-2.239661802466473 -1.5545673282960581 -2.44807600818014' if chirality == 'left' else '-2.239658800831686 -1.5545672668594075 -2.4480790171423275'}"/>
+         <geometry>
+            <mesh filename="${rospackage_path}/collision/tower_text_mesh.stl"/>
+         </geometry>
+         <material name="white"/>
+      </collision>
       <!-- Begin of extension modules-->
       <xacro:if value="${extension}">
@@ -68,5 +75,5 @@
       </visual>
       <collision name="collision_tower_fans_mesh">
-         <origin xyz="${s * 0.09363557490715463} -8.389280125979868e-05 0.007667379216642167" rpy="0.005482193788632295 ${s * 0.004072983473719427} -0.007158680095836076"/>
+         <origin xyz="${s * 0.09363557490715463} -8.389280125979868e-05 0.007667379216642167" rpy="0.005482193788632295 ${s * 0.004072983473719427} ${s * -0.007158680095836076}"/>
          <geometry>
             <mesh filename="${rospackage_path}/collision/tower_fans_mesh.stl"/>
@@ -75,5 +82,5 @@
       </collision>
       <visual name="visual_tower_u2d2_mesh">
-         <origin xyz="${s * -0.012411919130245945} 0.0016444826825456232 -0.017176262543363695" rpy="1.9248601461816697 0.03942618910803675 0.09532348749637565"/>
+         <origin xyz="${s * -0.012411919130245945} 0.0016444826825456232 -0.017176262543363695" rpy="1.9248601461816697 ${s * 0.03942618910803675} ${s * 0.09532348749637565}"/>
          <geometry>
             <mesh filename="${rospackage_path}/visual/tower_u2d2_mesh.stl"/>
@@ -82,5 +89,5 @@
       </visual>
       <collision name="collision_tower_u2d2_mesh">
-         <origin xyz=" ${s * -0.010637828550943964} 0.00323315623973064 -0.016564434073768834" rpy="1.9254973571203653 ${s * -0.010117808892087687} 0.1004013246446912"/>
+         <origin xyz=" ${s * -0.010637828550943964} 0.00323315623973064 -0.016564434073768834" rpy="1.9254973571203653 ${s * -0.010117808892087687} ${s * 0.1004013246446912}"/>
          <geometry>
             <mesh filename="${rospackage_path}/collision/tower_u2d2_mesh.stl"/>
@@ -114,19 +121,19 @@
       <parent link="${prefix}root"/>
       <child link="${prefix}world2tower_fixed_jointbody"/>
-      <origin xyz="${s * -0.0405} 0.0 0.05" rpy="0.0 0.0 0.0"/>
+      <origin xyz="${s * 0.04} 0.0 0.04575" rpy="0.0 0.0 0.0"/>
    </joint>
    <joint type="fixed" name="${prefix}world2tower_fixed_offset">
       <parent link="${prefix}world2tower_fixed_jointbody"/>
-      <child link="right_tower"/>
+      <child link="${prefix}tower"/>
       <origin xyz="-0.0 -0.0 -0.0" rpy="0.0 0.0 0.0"/>
    </joint>
    <link name="${prefix}palm">
       <inertial>
-         <origin xyz="${s * 0.00193} -0.00052 -0.00664" rpy="1.67519 0.04750000000000032 1.55556"/>
+         <origin xyz="${s * 0.00193} -0.00052 -0.00664" rpy="1.67519 ${s * 0.04750000000000032} ${s * 1.55556}"/>
          <mass value="0.0257"/>
          <inertia ixx="1.612e-05" iyy="1.151e-05" izz="6.72e-06" ixy="0" ixz="0" iyz="0"/>
       </inertial>
       <visual name="visual_palm_mesh">
-         <origin xyz="${s * 0.0015568393804010381} 0.00032366355975666324 -0.011896430343868667" rpy="${'-1.1152544578109254 0.044917456181218895 1.6097449018547754' if chirality == 'left' else '2.01172521777585 0.047179539585598285 1.531383022156099'}"/>
+         <origin xyz="${s * 0.0015568393804010381} 0.00032366355975666324 -0.011896430343868667" rpy="${'1.129867435813943 0.047179539585598285 1.6102096314336944' if chirality == 'left' else '2.01172521777585 0.047179539585598285 1.531383022156099'}"/>
          <geometry>
             <mesh filename="${rospackage_path}/visual/palm_mesh.stl"/>
@@ -135,5 +142,5 @@
       </visual>
       <collision name="right_collision_palm_mesh">
-         <origin xyz="0.0015796019462848588 0.0001376248446814945 -0.011923873250196919" rpy="2.026338195778868 0.044917456181218895 1.531847751735018"/>
+         <origin xyz="${s * 0.0015796019462848588} 0.0001376248446814945 -0.011923873250196919" rpy="${'1.1152544578109254 0.044917456181218895 1.6097449018547754' if chirality == 'left' else '2.026338195778868 0.044917456181218895 1.531847751735018'}"/>
          <geometry>
             <mesh filename="${rospackage_path}/collision/palm_mesh.stl"/>
@@ -142,5 +149,5 @@
       </collision>
       <visual name="right_visual_palm_skin_mesh">
-         <origin xyz="0.005673309514830851 -0.0012702684906836111 -0.001744430321194409" rpy="1.7666058493725336 0.1563942094199331 1.6505205003593353"/>
+         <origin xyz="${s * 0.005673309514830851} -0.0012702684906836111 -0.001744430321194409" rpy="${'1.3749868042172595 0.1563942094199331 1.4910721532304578' if chirality == 'left' else '1.7666058493725336 0.1563942094199331 1.6505205003593353'}"/>
          <geometry>
             <mesh filename="${rospackage_path}/visual/palm_skin_mesh.stl"/>
@@ -149,5 +156,5 @@
       </visual>
       <collision name="right_collision_palm_skin_mesh">
-         <origin xyz="0.008013832397891144 -0.001293701510845759 -0.0015696747425978242" rpy="1.8840619193629062 0.16785003095386486 1.6839920915628581"/>
+         <origin xyz="${s * 0.008013832397891144} -0.001293701510845759 -0.0015696747425978242" rpy="${'1.2575307342268869 0.16785003095386508 1.457600562026935' if chirality == 'left' else '1.8840619193629062 0.16785003095386486 1.6839920915628581'}"/>
          <geometry>
             <mesh filename="${rospackage_path}/collision/palm_skin_mesh.stl"/>
@@ -164,23 +171,23 @@
    </link>
    <joint type="revolute" name="right_wrist">
-      <parent link="right_tower"/>
+      <parent link="${prefix}tower"/>
       <child link="right_wrist_jointbody"/>
-      <origin xyz="0.04063 0.0 0.10486999999999999" rpy="0.0 0.0 0.0"/>
-      <axis xyz="1.0 0.0 0.0"/>
-      <limit lower="-0.6736" upper="0.8972" effort="100" velocity="100"/>
+      <origin xyz="${s * 0.04063} 0.0 0.10486999999999999" rpy="0.0 0.0 0.0"/>
+      <axis xyz="${s * 1.0} 0.0 0.0"/>
+      <limit lower="${-0.8972 if chirality == 'left' else -0.6736}" upper="${0.6736 if chirality == 'left' else 0.8972}" effort="100" velocity="100"/>
    </joint>
    <joint type="fixed" name="right_wrist_offset">
       <parent link="right_wrist_jointbody"/>
-      <child link="right_palm"/>
-      <origin xyz="-0.002 0.00144 0.03872" rpy="0.0 0.0 0.0"/>
+      <child link="${prefix}palm"/>
+      <origin xyz="${s * -0.002} 0.00144 0.03872" rpy="0.0 0.0 0.0"/>
    </joint>
    <link name="right_thumb_mp">
       <inertial>
-         <origin xyz="0.00247 0.0 0.004" rpy="0.0 0.016249999999999876 0.0"/>
+         <origin xyz="${s * 0.00247} 0.0 0.004" rpy="0.0 ${s * 0.016249999999999876} 0.0"/>
          <mass value="0.00586"/>
          <inertia ixx="8.4e-07" iyy="6.6e-07" izz="2.7e-07" ixy="0" ixz="0" iyz="0"/>
       </inertial>
       <visual name="right_visual_thumb_mp_mesh">
-         <origin xyz="0.0026672782758389094 -3.6617030073895996e-06 0.0032021510136003503" rpy="-0.00450638440425983 -0.0029041941261005455 0.0"/>
+         <origin xyz="${s * 0.0026672782758389094} -3.6617030073895996e-06 0.0032021510136003503" rpy="-0.00450638440425983 ${s * -0.0029041941261005455} 0.0"/>
          <geometry>
             <mesh filename="${rospackage_path}/visual/thumb_mp_mesh.stl"/>
@@ -189,5 +196,5 @@
       </visual>
       <collision name="right_collision_thumb_mp_mesh">
-         <origin xyz="0.0025186274059406416 1.1817094343651893e-05 0.0033325772179257306" rpy="-0.004051421860145692 0.0 0.0"/>
+         <origin xyz="${s * 0.0025186274059406416} 1.1817094343651893e-05 0.0033325772179257306" rpy="-0.004051421860145692 0.0 0.0"/>
          <geometry>
             <mesh filename="${rospackage_path}/collision/thumb_mp_mesh.stl"/>
@@ -204,7 +211,7 @@
    </link>
    <joint type="revolute" name="right_thumb_mcp">
-      <parent link="right_palm"/>
+      <parent link="${prefix}palm"/>
       <child link="right_thumb_mcp_jointbody"/>
-      <origin xyz="-0.02821 0.01777 -0.01321" rpy="0.5385700000000002 -0.05594999999999972 -1.27047"/>
+      <origin xyz="${s * -0.02821} 0.01777 -0.01321" rpy="0.5385700000000002 ${s * -0.05594999999999972} ${s * -1.27047}"/>
       <axis xyz="0.0 0.0 -1.0"/>
       <limit lower="-0.87266" upper="0.87266" effort="100" velocity="100"/>
@@ -217,10 +224,10 @@
    <link name="right_thumb_pp">
       <inertial>
-         <origin xyz="0.01848 1e-05 2e-05" rpy="1.5708 0.7739199999999999 1.5708"/>
+         <origin xyz="${s * 0.01848} 1e-05 2e-05" rpy="1.5708 ${s * 0.7739199999999999} ${s * 1.5708}"/>
          <mass value="0.00655"/>
          <inertia ixx="7.5e-07" iyy="7.1e-07" izz="3e-07" ixy="0" ixz="0" iyz="0"/>
       </inertial>
       <visual name="right_visual_thumb_pp_mesh">
-         <origin xyz="0.01772057472979195 1.0070925191614284e-05 -0.00010493568910233946" rpy="-1.6017800681828298 -1.1287165327427504 -1.5432562301164818"/>
+         <origin xyz="${s * 0.01772057472979195} 1.0070925191614284e-05 -0.00010493568910233946" rpy="${'-1.5398125854069626' if chirality == 'left' else '-1.6017800681828298'} -1.1287165327427504 ${'-1.5983364234733113' if chirality == 'left' else '-1.5432562301164818'}"/>
          <geometry>
             <mesh filename="${rospackage_path}/visual/thumb_pp_mesh.stl"/>
@@ -229,5 +236,5 @@
       </visual>
       <collision name="right_collision_thumb_pp_mesh">
-         <origin xyz="0.01727473106987278 2.0812531064334476e-05 -0.00010892038972696916" rpy="-1.588892025872152 -1.3512360913096229 -1.5473903377526785"/>
+         <origin xyz="${s * 0.01727473106987278} 2.0812531064334476e-05 -0.00010892038972696916" rpy="${'-1.552700627717642' if chirality == 'left' else '-1.588892025872152'} -1.3512360913096229 ${'-1.594202315837113' if chirality == 'left' else '-1.5473903377526785'}"/>
          <geometry>
             <mesh filename="${rospackage_path}/collision/thumb_pp_mesh.stl"/>
@@ -247,5 +254,5 @@
       <child link="right_thumb_abd_jointbody"/>
       <origin xyz="6.938893903907228e-18 0.0 0.0" rpy="-1.22173 0.0 0.0"/>
-      <axis xyz="0.0 0.34202085907197166 0.9396923602752502"/>
+      <axis xyz="0.0 ${s * 0.34202085907197166} ${s * 0.9396923602752502}"/>
       <limit lower="-1.08211" upper="0.0" effort="100" velocity="100"/>
    </joint>
@@ -253,14 +260,14 @@
       <parent link="right_thumb_abd_jointbody"/>
       <child link="right_thumb_pp"/>
-      <origin xyz="-0.03 -0.0 -0.0" rpy="0.0 0.0 0.0"/>
+      <origin xyz="${s * -0.03} -0.0 -0.0" rpy="0.0 0.0 0.0"/>
    </joint>
    <link name="right_thumb_ip">
       <inertial>
-         <origin xyz="0.00135 2e-05 0.01383" rpy="0.0003700000000000001 0.03263000000000016 0.00034"/>
+         <origin xyz="${s * 0.00135} 2e-05 0.01383" rpy="0.0003700000000000001 ${s * 0.03263000000000016} ${s * 0.00034}"/>
          <mass value="0.01402"/>
          <inertia ixx="1.7e-06" iyy="1.64e-06" izz="5.9e-07" ixy="0" ixz="0" iyz="0"/>
       </inertial>
       <visual name="right_visual_thumb_ip_mesh">
-         <origin xyz="0.0012998948492342203 7.159773213648307e-06 0.013619877706625217" rpy="0.0 0.04338716477372251 0.0"/>
+         <origin xyz="${s * 0.0012998948492342203} 7.159773213648307e-06 0.013619877706625217" rpy="0.0 0.04338716477372251 0.0"/>
          <geometry>
             <mesh filename="${rospackage_path}/visual/thumb_ip_mesh.stl"/>
@@ -269,5 +276,5 @@
       </visual>
       <collision name="right_collision_thumb_ip_mesh">
-         <origin xyz="0.0013560375396256981 0.00012710825491742077 0.013446327660739959" rpy="0.00708255798627546 0.04763590113115046 0.0"/>
+         <origin xyz="${s * 0.0013560375396256981} 0.00012710825491742077 0.013446327660739959" rpy="0.00708255798627546 0.04763590113115046 0.0"/>
          <geometry>
             <mesh filename="${rospackage_path}/collision/thumb_ip_mesh.stl"/>
@@ -276,5 +283,5 @@
       </collision>
       <visual name="right_visual_thumb_ip_skin_mesh">
-         <origin xyz="0.0015424443589898442 1.6522252825510055e-07 0.016259641785170875" rpy="3.141592653589793 -1.2480960827956862 0.0"/>
+         <origin xyz="${s * 0.0015424443589898442} 1.6522252825510055e-07 0.016259641785170875" rpy="${'0.0 -1.2480960827956862 3.141592653589793' if chirality == 'left' else '3.141592653589793 -1.2480960827956862 0.0'}"/>
          <geometry>
             <mesh filename="${rospackage_path}/visual/thumb_ip_skin_mesh.stl"/>
@@ -283,5 +290,5 @@
       </visual>
       <collision name="right_collision_thumb_ip_skin_mesh">
-         <origin xyz="0.0015528244655451595 6.48072440430664e-06 0.016246657621879965" rpy="3.141592653589793 -1.243771833702049 0.0"/>
+         <origin xyz="${s * 0.0015528244655451595} 6.48072440430664e-06 0.016246657621879965" rpy="${'0.0 -1.243771833702049 3.141592653589793' if chirality == 'left' else '3.141592653589793 -1.243771833702049 0.0'}"/>
          <geometry>
             <mesh filename="${rospackage_path}/collision/thumb_ip_skin_mesh.stl"/>
@@ -300,6 +307,6 @@
       <parent link="right_thumb_pp"/>
       <child link="right_thumb_pip_jointbody"/>
-      <origin xyz="0.0 0.0 0.0" rpy="-2.6535897934554242e-06 1.5707926535897934 3.141592653589793"/>
-      <axis xyz="0.0 -1.0 0.0"/>
+      <origin xyz="0.0 0.0 0.0" rpy="-2.6535897934554242e-06 ${s * 1.5707926535897934} 3.141592653589793"/>
+      <axis xyz="0.0 ${s * -1.0} 0.0"/>
       <limit lower="-0.7944" upper="1.23" effort="100" velocity="100"/>
    </joint>
@@ -316,5 +323,5 @@
       </inertial>
       <visual name="right_visual_thumb_dp_mesh">
-         <origin xyz="0.001737692119750562 -5.352917438125722e-06 0.005127321105400321" rpy="0.0 0.24698289481892632 0.0"/>
+         <origin xyz="${s * 0.001737692119750562} -5.352917438125722e-06 0.005127321105400321" rpy="0.0 ${s * 0.24698289481892632} 0.0"/>
          <geometry>
             <mesh filename="${rospackage_path}/visual/thumb_dp_mesh.stl"/>
@@ -323,5 +330,5 @@
       </visual>
       <collision name="right_collision_thumb_dp_mesh">
-         <origin xyz="0.0020244971365026335 3.68319791392775e-05 0.005533677984084769" rpy="0.24272423187789072 -0.008190712846545711 1.5687682825082248"/>
+         <origin xyz="${s * 0.0020244971365026335} 3.68319791392775e-05 0.005533677984084769" rpy="${s * 0.24272423187789072} -0.008190712846545711 ${'1.5728243710815684' if chirality == 'left' else '1.5687682825082248'}"/>
          <geometry>
             <mesh filename="${rospackage_path}/collision/thumb_dp_mesh.stl"/>
@@ -330,5 +337,5 @@
       </collision>
       <visual name="right_visual_thumb_dp_skin_mesh">
-         <origin xyz="0.002793435568551968 -6.14386555467744e-07 0.016601042013200628" rpy="3.141592653589793 -0.40239793279263236 0.0"/>
+         <origin xyz="${s * 0.002793435568551968} -6.14386555467744e-07 0.016601042013200628" rpy="${'0.0 -0.4023979327926315 3.141592653589793' if chirality == 'left' else '3.141592653589793 -0.40239793279263236 0.0'}"/>
          <geometry>
             <mesh filename="${rospackage_path}/visual/thumb_dp_skin_mesh.stl"/>
@@ -337,5 +344,5 @@
       </visual>
       <collision name="right_collision_thumb_dp_skin_mesh">
-         <origin xyz="0.002785448336058668 -6.944475247259374e-06 0.016557497442018437" rpy="3.141592653589793 -0.3963953079219906 0.0"/>
+         <origin xyz="${s * 0.002785448336058668} -6.944475247259374e-06 0.016557497442018437" rpy="${'0.0 -0.3963953079219906 3.141592653589793' if chirality == 'left' else '3.141592653589793 -0.3963953079219906 0.0'}"/>
          <geometry>
             <mesh filename="${rospackage_path}/collision/thumb_dp_skin_mesh.stl"/>
@@ -354,6 +361,6 @@
       <parent link="right_thumb_ip"/>
       <child link="right_thumb_dip_jointbody"/>
-      <origin xyz="0.0005 0.0 0.033" rpy="0.0 0.0 0.0"/>
-      <axis xyz="0.0 -1.0 0.0"/>
+      <origin xyz="${s * 0.0005} 0.0 0.033" rpy="0.0 0.0 0.0"/>
+      <axis xyz="0.0 ${s * -1.0} 0.0"/>
       <limit lower="-0.85384" upper="1.45" effort="100" velocity="100"/>
    </joint>
@@ -373,5 +380,5 @@
       <parent link="right_thumb_dp"/>
       <child link="right_thumb_fingertip"/>
-         <origin xyz="-0.003 0.0 0.025" rpy="0.0 0.0 0.0"/>
+         <origin xyz="${s * -0.003} 0.0 0.025" rpy="0.0 0.0 0.0"/>
    </joint>
    <link name="right_index_mp">
@@ -382,5 +389,5 @@
       </inertial>
       <visual name="right_visual_index_mp_mesh">
-         <origin xyz="0.010698479000335614 -1.389065483476104e-05 -0.00027878809319396305" rpy="3.1297715721932393 -1.5066740246432395 2.4424906541753444e-15"/>
+         <origin xyz="${'-0.010698479000335614 -1.3890654834761171e-05 -0.00027878809319396294' if chirality == 'left' else '0.010698479000335614 -1.389065483476104e-05 -0.00027878809319396305'}" rpy="${'0.011821081396553579' if chirality == 'left' else '3.1297715721932393'} -1.5066740246432395 ${'3.1415926535897905' if chirality == 'left' else '2.4424906541753444e-15'}"/>
          <geometry>
             <mesh filename="${rospackage_path}/visual/index_mp_mesh.stl"/>
@@ -389,5 +396,5 @@
       </visual>
       <collision name="right_collision_index_mp_mesh">
-         <origin xyz="0.01047824184159959 -4.456734197189478e-05 -0.00016480462181888062" rpy="0.928212641576985 -1.5147947849129795 2.212627507721145"/>
+         <origin xyz="${'-0.01047824184159959 -4.456734197189497e-05 -0.00016480462181888051' if chirality == 'left' else '0.01047824184159959 -4.456734197189478e-05 -0.00016480462181888062'}" rpy="${'2.2133800120128084' if chirality == 'left' else '0.928212641576985'} -1.5147947849129795 ${'0.9289651458686482' if chirality == 'left' else '2.212627507721145'}"/>
          <geometry>
             <mesh filename="${rospackage_path}/collision/index_mp_mesh.stl"/>
@@ -404,8 +411,8 @@
    </link>
    <joint type="revolute" name="right_index_abd">
-      <parent link="right_palm"/>
+      <parent link="${prefix}palm"/>
       <child link="right_index_abd_jointbody"/>
-      <origin xyz="-0.024088797002689358 0.0018999642829399502 0.025164928786148736" rpy="1.6066999999999996 1.13552 -0.05339000000000049"/>
-      <axis xyz="0.0 0.0 -1.0"/>
+      <origin xyz="${s * -0.024088797002689358} 0.0018999642829399502 0.025164928786148736" rpy="1.6066999999999996 ${s * 1.13552} ${s * -0.05339000000000049}"/>
+      <axis xyz="0.0 0.0 ${s * -1.0}"/>
       <limit lower="-1.04577" upper="0.24577" effort="100" velocity="100"/>
    </joint>
@@ -413,14 +420,14 @@
       <parent link="right_index_abd_jointbody"/>
       <child link="right_index_mp"/>
-      <origin xyz="-0.02 -0.0 -0.0" rpy="0.0 0.0 0.0"/>
+      <origin xyz="${s * -0.02} -0.0 -0.0" rpy="0.0 0.0 0.0"/>
    </joint>
    <link name="right_index_pp">
       <inertial>
-         <origin xyz="0.00135 2e-05 0.01637" rpy="0.00034 0.020550000000000068 0.00038"/>
+         <origin xyz="${s * 0.00135} 2e-05 0.01637" rpy="0.00034 ${s * 0.020550000000000068} ${s * 0.00038}"/>
          <mass value="0.0165"/>
          <inertia ixx="2.39e-06" iyy="2.31e-06" izz="7.1e-07" ixy="0" ixz="0" iyz="0"/>
       </inertial>
       <visual name="right_visual_index_pp_mesh">
-         <origin xyz="0.0012791981098529209 4.322204569499314e-05 0.016098661080179" rpy="0.005516325755706635 0.035101984887858206 0.03910570256058449"/>
+         <origin xyz="${s * 0.0012791981098529209} 4.322204569499314e-05 0.016098661080179" rpy="0.005516325755706635 ${s * 0.035101984887858206} ${s * 0.03910570256058449}"/>
          <geometry>
             <mesh filename="${rospackage_path}/visual/index_pp_mesh.stl"/>
@@ -429,5 +436,5 @@
       </visual>
       <collision name="right_collision_index_pp_mesh">
-         <origin xyz="0.0013516740131344841 1.1247422892215125e-05 0.015681803525061735" rpy="0.0 0.042883356216690816 0.0"/>
+         <origin xyz="${s * 0.0013516740131344841} 1.1247422892215125e-05 0.015681803525061735" rpy="0.0 ${s * 0.042883356216690816} 0.0"/>
          <geometry>
             <mesh filename="${rospackage_path}/collision/index_pp_mesh.stl"/>
@@ -436,5 +443,5 @@
       </collision>
       <visual name="right_visual_index_pp_skin_mesh">
-         <origin xyz="0.0016617007377281573 7.13567847691717e-08 0.018763861638214734" rpy="3.141592653589793 -0.8345404465359767 0.0"/>
+         <origin xyz="${s * 0.0016617007377281573} 7.13567847691717e-08 0.018763861638214734" rpy="${'0.0 -0.8345404465359767 3.141592653589793' if chirality == 'left' else '3.141592653589793 -0.8345404465359767 0.0'}"/>
          <geometry>
             <mesh filename="${rospackage_path}/visual/index_pp_skin_mesh.stl"/>
@@ -443,5 +450,5 @@
       </visual>
       <collision name="right_collision_index_pp_skin_mesh">
-         <origin xyz="0.0016773866527582534 -5.5310131701629075e-06 0.018740870134460883" rpy="3.141592653589793 -0.8259683678608123 0.0"/>
+         <origin xyz="${s * 0.0016773866527582534} -5.5310131701629075e-06 0.018740870134460883" rpy="${'0.0 -0.8259683678608112 3.141592653589793' if chirality == 'left' else '3.141592653589793 -0.8259683678608123 0.0'}"/>
          <geometry>
             <mesh filename="${rospackage_path}/collision/index_pp_skin_mesh.stl"/>
@@ -460,6 +467,6 @@
       <parent link="right_index_mp"/>
       <child link="right_index_mcp_jointbody"/>
-      <origin xyz="0.0 0.0 0.0" rpy="3.141592653589793 -1.5707926535897931 3.141592653589793"/>
-      <axis xyz="0.0 -1.0 0.0"/>
+      <origin xyz="0.0 0.0 0.0" rpy="3.141592653589793 ${s * -1.5707926535897931} 3.141592653589793"/>
+      <axis xyz="0.0 ${s * -1.0} 0.0"/>
       <limit lower="-0.34907" upper="1.65806" effort="100" velocity="100"/>
    </joint>
@@ -471,10 +478,10 @@
    <link name="right_index_ip">
       <inertial>
-         <origin xyz="0.00071 1e-05 0.01929" rpy="-0.00042000000000000023 -0.18548999999999993 0.004400000000000001"/>
+         <origin xyz="${s * 0.00071} 1e-05 0.01929" rpy="-0.00042000000000000023 ${s * -0.18548999999999993} ${s * 0.004400000000000001}"/>
          <mass value="0.01521"/>
          <inertia ixx="2.08e-06" iyy="2.06e-06" izz="5.4e-07" ixy="0" ixz="0" iyz="0"/>
       </inertial>
       <visual name="right_visual_index_ip_mesh">
-         <origin xyz="0.0010416798025929732 7.836534536637715e-05 0.011793743862640304" rpy="-0.03448776902850714 -0.0034390239986910043 1.5709149778710771"/>
+         <origin xyz="${s * 0.0010416798025929732} 7.836534536637715e-05 0.011793743862640304" rpy="${s * -0.03448776902850714} -0.0034390239986910043 ${'1.5706776757187162' if chirality == 'left' else '1.5709149778710771'}"/>
          <geometry>
             <mesh filename="${rospackage_path}/visual/index_ip_mesh.stl"/>
@@ -483,5 +490,5 @@
       </visual>
       <collision name="right_collision_index_ip_mesh">
-         <origin xyz="0.001264526142413497 -1.637119615337525e-05 0.01147202326458154" rpy="0.0018005943049513862 0.0 1.5707963267948966"/>
+         <origin xyz="${s * 0.001264526142413497} -1.637119615337525e-05 0.01147202326458154" rpy="${s * 0.0018005943049513862} 0.0 1.5707963267948966"/>
          <geometry>
             <mesh filename="${rospackage_path}/collision/index_ip_mesh.stl"/>
@@ -490,5 +497,5 @@
       </collision>
       <visual name="right_visual_index_ip_skin_mesh">
-         <origin xyz="0.0006177579160319044 -2.8394632435300543e-07 0.02298191534250252" rpy="0.0 -0.4563594541722644 0.0"/>
+         <origin xyz="${s * 0.0006177579160319044} -2.8394632435300543e-07 0.02298191534250252" rpy="0.0 ${s * -0.4563594541722644} 0.0"/>
          <geometry>
             <mesh filename="${rospackage_path}/visual/index_ip_skin_mesh.stl"/>
@@ -497,5 +504,5 @@
       </visual>
       <collision name="right_collision_index_ip_skin_mesh">
-         <origin xyz="0.0006216739383467692 2.432607491983251e-06 0.02302104994067657" rpy="0.0 -0.4457042297154219 0.0"/>
+         <origin xyz="${s * 0.0006216739383467692} 2.432607491983251e-06 0.02302104994067657" rpy="0.0 ${s * -0.4457042297154219} 0.0"/>
          <geometry>
             <mesh filename="${rospackage_path}/collision/index_ip_skin_mesh.stl"/>
@@ -514,6 +521,6 @@
       <parent link="right_index_pp"/>
       <child link="right_index_pip_jointbody"/>
-      <origin xyz="0.0005 0.0 0.038" rpy="0.0 0.0 0.0"/>
-      <axis xyz="0.0 -1.0 0.0"/>
+      <origin xyz="${s * 0.0005} 0.0 0.038" rpy="0.0 0.0 0.0"/>
+      <axis xyz="0.0 ${s * -1.0} 0.0"/>
       <limit lower="-0.34907" upper="1.88496" effort="100" velocity="100"/>
    </joint>
@@ -533,5 +540,5 @@
       <parent link="right_index_ip"/>
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