Commit message: organize stl files accordingly

File: models/urdf/orcahand.urdf.xacro (robot description, xacro)
@@ -9,5 +9,5 @@
   <xacro:property name="chirality" value="$(arg chirality)"/>
   <xacro:property name="s" value="${-1 if chirality == 'left' else 1}"/>
-  <xacro:property name="rospackage_path" value="package://orcahand_description/assets/urdf/right"/>
+  <xacro:property name="rospackage_path" value="package://orcahand_description/assets/urdf"/>
    <link name="${prefix}root">
       <inertial>
@@ -26,5 +26,5 @@
          <origin xyz="${s * 0.04069509610470536} -0.00012511806280993186 0.02312294830988657" rpy="-0.007252153364137093 ${s * -0.004356332895580239} ${s * 1.533990149039079}"/>
          <geometry>
-            <mesh filename="package://orcahand_description/assets/urdf/right/visual/tower_main_mesh.stl"
+            <mesh filename="package://orcahand_description/assets/urdf/visual/tower_main_mesh.stl"
                   scale="${'-1 1 1' if chirality == 'left' else '1 1 1'}"
             />
@@ -118,5 +118,5 @@
          <origin xyz="${s * 0.04141561887638722} 0.052825801794652016 -0.019856742052109723" rpy="-3.066013393320364 ${s * -1.0811766886677918} ${s * -1.6762365509261419}"/>
          <geometry>
-            <mesh filename="package://orcahand_description/assets/urdf/right/visual/tower_camera_mesh.stl"
+            <mesh filename="package://orcahand_description/assets/urdf/visual/tower_camera_mesh.stl"
              scale="${'-1 1 1' if chirality == 'left' else '1 1 1'}"/>
          </geometry>
@@ -432,5 +432,5 @@
       </inertial>
    </link>
-   <joint type="fixed" name="thumb_dp2right_thumb_fingertip_fixed_offset">
+   <joint type="fixed" name="${prefix}thumb_dp2thumb_fingertip_fixed_offset">
       <parent link="${prefix}thumb_dp"/>
       <child link="${prefix}thumb_fingertip"/>
@@ -612,5 +612,5 @@
       </inertial>
    </link>
-   <joint type="fixed" name="${prefix}index_ip2right_index_fingertip_fixed_offset">
+   <joint type="fixed" name="${prefix}index_ip2index_fingertip_fixed_offset">
       <parent link="${prefix}index_ip"/>
       <child link="${prefix}index_fingertip"/>
@@ -792,5 +792,5 @@
       </inertial>
    </link>
-   <joint type="fixed" name="${prefix}middle_ip2right_index_fingertip_fixed_offset">
+   <joint type="fixed" name="${prefix}middle_ip2middle_fingertip_fixed_offset">
       <parent link="${prefix}middle_ip"/>
       <child link="${prefix}middle_fingertip"/>
@@ -972,5 +972,5 @@
       </inertial>
    </link>
-   <joint type="fixed" name="${prefix}ring_ip2right_index_fingertip_fixed_offset">
+   <joint type="fixed" name="${prefix}ring_ip2ring_fingertip_fixed_offset">
       <parent link="${prefix}ring_ip"/>
       <child link="${prefix}ring_fingertip"/>
@@ -1152,5 +1152,5 @@
       </inertial>
    </link>
-   <joint type="fixed" name="${prefix}pinky_ip2right_index_fingertip_fixed_offset">
+   <joint type="fixed" name="${prefix}pinky_ip2pinky_fingertip_fixed_offset">
       <parent link="${prefix}pinky_ip"/>
       <child link="${prefix}pinky_fingertip"/>

Commit message: debug the range limits in urdf xacro

File: models/urdf/orcahand.urdf.xacro (robot description, xacro)
@@ -206,5 +206,5 @@
       <origin xyz="${s * 0.04063} 0.0 0.10486999999999999" rpy="0.0 0.0 0.0"/>
       <axis xyz="1.0 0.0 0.0"/>
-      <limit lower="${-0.8972 if chirality == 'left' else -0.6736}" upper="${0.6736 if chirality == 'left' else 0.8972}" effort="100" velocity="100"/>
+      <limit lower="-0.872665" upper="0.523599" effort="100" velocity="100"/>
    </joint>
    <joint type="fixed" name="${prefix}wrist_offset">
@@ -294,5 +294,5 @@
       <origin xyz="6.938893903907228e-18 0.0 0.0" rpy="-1.22173 0.0 0.0"/>
       <axis xyz="0.0 ${s * 0.34202085907197166} ${s * 0.9396923602752502}"/>
-      <limit lower="-1.08211" upper="0.0" effort="100" velocity="100"/>
+      <limit lower="-0.349066" upper="0.733038" effort="100" velocity="100"/>
    </joint>
    <joint type="fixed" name="${prefix}thumb_abd_offset">
@@ -356,5 +356,5 @@
       <origin xyz="0.0 0.0 0.0" rpy="-2.6535897934554242e-06 ${s * 1.5707926535897934} ${s * 3.141592653589793}"/>
       <axis xyz="0.0 ${s * -1.0} 0.0"/>
-      <limit lower="-0.7944" upper="1.23" effort="100" velocity="100"/>
+      <limit lower="-0.209440" upper="1.884956" effort="100" velocity="100"/>
    </joint>
    <joint type="fixed" name="${prefix}thumb_pip_offset">
@@ -418,5 +418,5 @@
       <origin xyz="${s * 0.0005} 0.0 0.033" rpy="0.0 0.0 0.0"/>
       <axis xyz="0.0 ${s * -1.0} 0.0"/>
-      <limit lower="-0.85384" upper="1.45" effort="100" velocity="100"/>
+      <limit lower="-0.349066" upper="1.954769" effort="100" velocity="100"/>
    </joint>
    <joint type="fixed" name="${prefix}thumb_dip_offset">
@@ -474,5 +474,5 @@
       <origin xyz="${s * -0.024088797002689358} 0.0018999642829399502 0.025164928786148736" rpy="1.6066999999999996 ${s * 1.13552} ${s * -0.05339000000000049}"/>
       <axis xyz="0.0 0.0 ${s * -1.0}"/>
-      <limit lower="-1.04577" upper="0.24577" effort="100" velocity="100"/>
+      <limit lower="-0.645772" upper="0.645772" effort="100" velocity="100"/>
    </joint>
    <joint type="fixed" name="${prefix}index_abd_offset">
@@ -536,5 +536,5 @@
       <origin xyz="0.0 0.0 0.0" rpy="3.141592653589793 ${s * -1.5707926535897931} ${s * 3.141592653589793}"/>
       <axis xyz="0.0 ${s * -1.0} 0.0"/>
-      <limit lower="-0.34907" upper="1.65806" effort="100" velocity="100"/>
+      <limit lower="-0.349066" upper="1.658063" effort="100" velocity="100"/>
    </joint>
    <joint type="fixed" name="${prefix}index_mcp_offset">
@@ -598,5 +598,5 @@
       <origin xyz="${s * 0.0005} 0.0 0.038" rpy="0.0 0.0 0.0"/>
       <axis xyz="0.0 ${s * -1.0} 0.0"/>
-      <limit lower="-0.34907" upper="1.88496" effort="100" velocity="100"/>
+      <limit lower="-0.349066" upper="1.884956" effort="100" velocity="100"/>
    </joint>
    <joint type="fixed" name="${prefix}index_pip_offset">
@@ -654,5 +654,5 @@
       <origin xyz="${s * -7.346410206776621e-08} 0.0 0.030000000000134926" rpy="-1.5707926536208807 ${s * 1.5707926535897934} ${s * 3.141592653558706}"/>
       <axis xyz="0.0 0.0 ${s * -1.0}"/>
-      <limit lower="-0.64577" upper="0.64577" effort="100" velocity="100"/>
+      <limit lower="-0.645772" upper="0.645772" effort="100" velocity="100"/>
    </joint>
    <joint type="fixed" name="${prefix}middle_abd_offset">
@@ -716,5 +716,5 @@
       <origin xyz="0.0 0.0 0.0" rpy="3.141592653589793 ${s * -1.5707926535897931} ${s * 3.141592653589793}"/>
       <axis xyz="0.0 ${s * -1.0} 0.0"/>
-      <limit lower="-0.34907" upper="1.58825" effort="100" velocity="100"/>
+      <limit lower="-0.349066" upper="1.588250" effort="100" velocity="100"/>
    </joint>
    <joint type="fixed" name="${prefix}middle_mcp_offset">
@@ -778,5 +778,5 @@
       <origin xyz="${s * 0.0005} 0.0 0.046" rpy="0.0 0.0 0.0"/>
       <axis xyz="0.0 ${s * -1.0} 0.0"/>
-      <limit lower="-0.34907" upper="1.8675" effort="100" velocity="100"/>
+      <limit lower="-0.349066" upper="1.867502"  effort="100" velocity="100"/>
    </joint>
    <joint type="fixed" name="${prefix}middle_pip_offset">
@@ -834,5 +834,5 @@
       <origin xyz="${s * 0.021521022061295733} 0.0015382095479525787 0.020824784431525818" rpy="-1.5359699999999998 ${s * 1.30836} ${s * -3.05441}"/>
       <axis xyz="0.0 0.0 ${s * -1.0}"/>
-      <limit lower="-0.47577" upper="0.80577" effort="100" velocity="100"/>
+      <limit lower="-0.645772" upper="0.645772"  effort="100" velocity="100"/>
    </joint>
    <joint type="fixed" name="${prefix}ring_abd_offset">
@@ -896,5 +896,5 @@
       <origin xyz="0.0 0.0 0.0" rpy="3.141592653589793 ${s * -1.5707926535897931} ${s * 3.141592653589793}"/>
       <axis xyz="0.0 ${s * -1.0} 0.0"/>
-      <limit lower="-0.34907" upper="1.58825" effort="100" velocity="100"/>
+      <limit lower="-0.349066" upper="1.588250"  effort="100" velocity="100"/>
    </joint>
    <joint type="fixed" name="${prefix}ring_mcp_offset">
@@ -958,5 +958,5 @@
       <origin xyz="${s * 0.0005} 0.0 0.046" rpy="0.0 0.0 0.0"/>
       <axis xyz="0.0 ${s * -1.0} 0.0"/>
-      <limit lower="-0.34907" upper="1.8675" effort="100" velocity="100"/>
+      <limit lower="-0.349066" upper="1.867502"  effort="100" velocity="100"/>
    </joint>
    <joint type="fixed" name="${prefix}ring_pip_offset">
@@ -1014,5 +1014,5 @@
       <origin xyz="${s * 0.04258452932438962} 0.004988143142003794 0.007243722937596895" rpy="-1.49694 ${s * 0.8614899999999999} ${s * -2.8837299999999995}"/>
       <axis xyz="0.0 0.0 ${s * -1.0}"/>
-      <limit lower="-0.12244" upper="1.1691" effort="100" velocity="100"/>
+      <limit lower="-0.645772" upper="0.645772"  effort="100" velocity="100"/>
    </joint>
    <joint type="fixed" name="${prefix}pinky_abd_offset">
@@ -1076,5 +1076,5 @@
       <origin xyz="0.0 0.0 0.0" rpy="3.141592653589793 ${s * -1.5707926535897931} ${s * 3.141592653589793}"/>
       <axis xyz="0.0 ${s * -1.0} 0.0"/>
-      <limit lower="-0.34907" upper="1.71042" effort="100" velocity="100"/>
+      <limit lower="-0.349066" upper="1.710423" effort="100" velocity="100"/>
    </joint>
    <joint type="fixed" name="${prefix}pinky_mcp_offset">
@@ -1138,5 +1138,5 @@
       <origin xyz="${s * 0.0005} 0.0 0.033" rpy="0.0 0.0 0.0"/>
       <axis xyz="0.0 ${s * -1.0} 0.0"/>
-      <limit lower="-0.34907" upper="1.88496" effort="100" velocity="100"/>
+      <limit lower="-0.349066" upper="1.884956" effort="100" velocity="100"/>
    </joint>
    <joint type="fixed" name="${prefix}pinky_pip_offset">

Commit message: amend

File: models/urdf/orcahand.urdf.xacro (robot description, xacro)
@@ -26,5 +26,5 @@
          <origin xyz="${s * 0.04069509610470536} -0.00012511806280993186 0.02312294830988657" rpy="-0.007252153364137093 ${s * -0.004356332895580239} ${s * 1.533990149039079}"/>
          <geometry>
-            <mesh filename="package://orcahand_description/assets/urdf/visual/tower_main_mesh.stl"
+            <mesh filename="${rospackage_path}/visual/tower_main_mesh.stl"
                   scale="${'-1 1 1' if chirality == 'left' else '1 1 1'}"
             />
@@ -118,5 +118,5 @@
          <origin xyz="${s * 0.04141561887638722} 0.052825801794652016 -0.019856742052109723" rpy="-3.066013393320364 ${s * -1.0811766886677918} ${s * -1.6762365509261419}"/>
          <geometry>
-            <mesh filename="package://orcahand_description/assets/urdf/visual/tower_camera_mesh.stl"
+            <mesh filename="${rospackage_path}/visual/tower_camera_mesh.stl"
              scale="${'-1 1 1' if chirality == 'left' else '1 1 1'}"/>
          </geometry>
